File: PCB_Schema/Drifter.kicad_pcb (KiCad board)
At the start: 2 copper layers, 11 parts, among them J2 PinSocket_1x04_P2.54mm_Vertic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, U1 Max6675, U2 74VHC125, U3 DHT11, U4 LM3940

Commit message: Updated KiCad PCB/Schema files
Parts:
- removed A1: Arduino_UNO_R3, Module:Arduino_UNO_R3
- added J3: 2-Terminal Wire-to-board, DrifterLibrary:2-Terminal Wire-to-board, F.Cu at (205.2, 66.4)
- added J3: PinHeader_1x02_P2.54mm_Vertical, Connector_PinHeader_2.54mm:PinHeader_1x02_P2.54mm_Vertical, F.Cu at (176.3, 48.8)
- added J4: PinHeader_1x02_P2.54mm_Vertical, Connector_PinHeader_2.54mm:PinHeader_1x02_P2.54mm_Vertical, F.Cu at (180.8, 56.3)
- added J5: PinHeader_1x05_P2.54mm_Vertical, Connector_PinHeader_2.54mm:PinHeader_1x05_P2.54mm_Vertical, F.Cu at (176.1, 61.0)
- added J6: PinHeader_1x02_P2.54mm_Vertical, Connector_PinHeader_2.54mm:PinHeader_1x02_P2.54mm_Vertical, F.Cu at (190.7, 60.8)
- added J7: PinHeader_1x02_P2.54mm_Vertical, Connector_PinHeader_2.54mm:PinHeader_1x02_P2.54mm_Vertical, F.Cu at (176.0, 77.7)
- added J8: PinHeader_1x02_P2.54mm_Vertical, Connector_PinHeader_2.54mm:PinHeader_1x02_P2.54mm_Vertical, F.Cu at (174.5, 84.1)
- added J9: PinHeader_1x02_P2.54mm_Vertical, Connector_PinHeader_2.54mm:PinHeader_1x02_P2.54mm_Vertical, F.Cu at (185.8, 105.7)
- added Power In: PinHeader_1x02_P2.54mm_Vertical, Connector_PinHeader_2.54mm:PinHeader_1x02_P2.54mm_Vertical, F.Cu at (165.1, 105.4)
- C1, C2: value 100nF -> C_0603_1608Metric; footprint Capacitor_SMD:C_01005_0402Metric -> Capacitor_SMD:C_0603_1608Metric
- U3: value DHT11 -> Aosong_DHT11_5.5x12.0_P2.54mm
- moved U3 72.2 mm to (198.3, 76.6), turned to 0 degrees
- moved C4 68.2 mm to (172.8, 107.7), turned to 180 degrees
- moved U4 59.6 mm to (169.6, 86.4), turned to 0 degrees
- moved J2 56.9 mm to (189.2, 53.7), turned to 180 degrees
- moved C3 56.3 mm to (176.3, 108.5), turned to 180 degrees
- moved U1 5.21 mm to (195.5, 66.3)
- moved C1 4.02 mm to (199.4, 62.2), turned to 0 degrees
- moved C2 2.97 mm to (190.5, 91.4), turned to 0 degrees
- renumbered REF** to J1
Connections:
- C1 pad 1: (no net) -> +5V
- C1 pad 2: (no net) -> GND
- C3 pad 1: (no net) -> +3.3V
- C3 pad 2: (no net) -> GND
- C4 pad 1: (no net) -> GND
- C4 pad 2: (no net) -> +5V
- J2 pad 1: (no net) -> +5V
- J2 pad 2: (no net) -> RX
- J2 pad 3: (no net) -> TX
- J2 pad 4: (no net) -> GND
- U1 pad 1: (no net) -> GND
- U1 pad 2: (no net) -> T-
- U1 pad 3: (no net) -> T+
- U1 pad 4: (no net) -> +5V
- U1 pad 5: (no net) -> /SCK
- U1 pad 6: (no net) -> /CS_Thermo
- U1 pad 7: (no net) -> /MISO
- U3 pad 2: Net-(A1-Pad17) -> IO
- U3 pad 3: unconnected-(U3-Pad3) -> (no net)
- U4 pad 1: (no net) -> +5V
- U4 pad 2: (no net) -> GND
- U4 pad 3: (no net) -> +3.3V
Routing:
- net +5V: track 0.00 -> 133.5 mm, vias 0 -> 1
- net +3.3V: track 3.23 -> 65.0 mm, vias 0 -> 1
- net /MISO: track 13.5 -> 65.7 mm, vias 2 -> 5
- net /SCK: track 22.9 -> 59.8 mm, vias 0 -> 2
- net /CS_SD: track 16.8 -> 48.8 mm
- net /MOSI: track 16.0 -> 40.9 mm, vias 0 -> 2
- net IO: track 0.00 -> 23.6 mm, vias 0 -> 2
- net /CS_Thermo: track 0.00 -> 18.2 mm
- net GND: track 3.29 -> 20.6 mm, vias 0 -> 1
- net TX: track 0.00 -> 13.0 mm
- net RX: track 0.00 -> 13.0 mm
- net T-: track 0.00 -> 8.26 mm
- net T+: track 0.00 -> 8.16 mm
- added copper zone on B.Cu, net GND
- added copper zone on F.Cu, net GND
Other:
- board outline added: 53.3 x 76.2 mm
- board text added: "DHT 11: Data -> GND ->"
- board text added: "GND +5V"
- board text added: "GPS: TX -> RX ->"
- board text added: "OSU Ocean Drifter Kit Breakout Board V1.0 Designed by Austin Green"
- board text added: "SPI: SCK -> MISO -> MOSI -> Thermo_CS-> SD_CS ->"

Commit message: Updated PCB
Parts:
- removed J5: PinHeader_1x05_P2.54mm_Vertical, Connector_PinHeader_2.54mm:PinHeader_1x05_P2.54mm_Vertical
- removed J7: PinHeader_1x02_P2.54mm_Vertical, Connector_PinHeader_2.54mm:PinHeader_1x02_P2.54mm_Vertical
- removed U3: Aosong_DHT11_5.5x12.0_P2.54mm, Sensor:Aosong_DHT11_5.5x12.0_P2.54mm
- added C5: C_0805_2012Metric, Capacitor_SMD:C_0805_2012Metric, F.Cu at (73.2, 105.2)
- added GPS_Power: LED_0805_2012Metric, LED_SMD:LED_0805_2012Metric, F.Cu at (76.7, 45.2)
- added Main_Power: LED_0805_2012Metric, LED_SMD:LED_0805_2012Metric, F.Cu at (75.7, 115.6)
- added R1: R_0805_2012Metric, Resistor_SMD:R_0805_2012Metric, F.Cu at (82.5, 45.2)
- added R2: R_0805_2012Metric, Resistor_SMD:R_0805_2012Metric, F.Cu at (81.6, 54.1)
- added R3: R_0805_2012Metric, Resistor_SMD:R_0805_2012Metric, F.Cu at (79.1, 81.0)
- added R4: R_0805_2012Metric, Resistor_SMD:R_0805_2012Metric, F.Cu at (88.9, 107.2)
- added R5: R_0805_2012Metric, Resistor_SMD:R_0805_2012Metric, F.Cu at (81.3, 115.6)
- added SD_Power: LED_0805_2012Metric, LED_SMD:LED_0805_2012Metric, F.Cu at (83.8, 107.2)
- added T1: PinHeader_1x02_P2.54mm_Vertical, Connector_PinHeader_2.54mm:PinHeader_1x02_P2.54mm_Vertical, F.Cu at (104.7, 61.9)
- added T1_Power: LED_0805_2012Metric, LED_SMD:LED_0805_2012Metric, F.Cu at (75.7, 54.1)
- added T2: Max6675, DrifterLibrary:Max6675, F.Cu at (92.0, 70.0)
- added T2: PinHeader_1x02_P2.54mm_Vertical, Connector_PinHeader_2.54mm:PinHeader_1x02_P2.54mm_Vertical, F.Cu at (104.7, 68.8)
- added T2_Power: LED_0805_2012Metric, LED_SMD:LED_0805_2012Metric, F.Cu at (73.2, 81.0)
- C1, C2: value C_0603_1608Metric -> C_0805_2012Metric; footprint Capacitor_SMD:C_0603_1608Metric -> Capacitor_SMD:C_0805_2012Metric
- C4: value C_0201_0603Metric -> C_0805_2012Metric; footprint Capacitor_SMD:C_0201_0603Metric -> Capacitor_SMD:C_0805_2012Metric
- J3: value 2-Terminal Wire-to-board -> PinHeader_1x06_P2.54mm_Vertical; footprint DrifterLibrary:2-Terminal Wire-to-board -> Connector_PinHeader_2.54mm:PinHeader_1x06_P2.54mm_Vertical
- moved J3 133.1 mm to (72.5, 57.8), turned to 0 degrees
- moved P2 115.6 mm to (75.7, 49.5)
- moved J1 106.3 mm to (71.1, 33.4)
- moved J2 106.3 mm to (84.0, 38.3)
- moved P1 106.3 mm to (75.7, 40.9)
- moved T1 103.4 mm to (92.1, 63.2)
- moved J1 103.4 mm to (99.9, 93.4)
- moved P4 103.4 mm to (82.5, 102.5)
- moved U4 103.4 mm to (66.3, 83.3)
- moved C4 103.3 mm to (69.6, 105.2), turned to 0 degrees
- moved C1 103.2 mm to (96.3, 58.9)
- moved P3 102.5 mm to (72.4, 75.7)
- moved U2 102.2 mm to (83.3, 93.4)
- moved Power In 99.6 mm to (66.0, 115.3)
- moved C2 94.5 mm to (99.3, 66.8)
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- renumbered J3 to J1, J4 to P1, J6 to P2, J8 to P3, J9 to P4, U1 to T1
Connections:
- C2 pad 1: +3.3V -> +5V
- C4 pad 1: GND -> +5V
- C4 pad 2: +5V -> GND
- J3 pad 1: T- -> /SCK
- J3 pad 2: T+ -> /MISO
Routing:
- net +5V: track 133.5 -> 199.1 mm, vias 1 -> 3
- net IO: track 23.6 -> 0.00 mm, vias 2 -> 0
- net (no net): track 0.00 -> 20.6 mm
- net GND: track 20.6 -> 39.7 mm, vias 1 -> 2
- net CS_Thermo2: track 0.00 -> 17.8 mm
- net /SCK: track 59.8 -> 70.9 mm, vias 2 -> 3
- net T2+: track 0.00 -> 10.6 mm
- net T2-: track 0.00 -> 10.6 mm
- net +3.3V: track 65.0 -> 71.9 mm
- net /MISO: track 65.7 -> 71.9 mm, vias 5 -> 6
- net T+: track 8.16 -> 10.5 mm
- net T-: track 8.26 -> 10.5 mm
- net CD: track 21.8 -> 23.0 mm
- net /MOSI: track 40.9 -> 41.7 mm
Other:
- board size 53.3 x 76.2 mm -> 61 x 101.6 mm
- board text added: "+"
- board text added: "-"
- board text added: "OSU Ocean Drifter Kit Breakout Board V1.2 Designed by Austin Green"
- board text added: "SD Card"
- board text added: "SPI: SCK -> MISO -> MOSI -> Thermo_CS-> Thermo_CS2-> SD_CS ->"
- board text added: "Thermocouples"
- board text removed: "DHT 11: Data -> GND ->"
- board text removed: "OSU Ocean Drifter Kit Breakout Board V1.0 Designed by Austin Green"
- board text removed: "SPI: SCK -> MISO -> MOSI -> Thermo_CS-> SD_CS ->"
